File: boardFiles/BoardVariant/solution/schematic.brd (EAGLE design)
At the start: 88.6 x 63.5 mm, 4 parts, among them IC1 MSP430F1491, IC2 BQ24120

Commit message: Normal Push.
Parts:
- removed IC2: BQ24120, texas:QFN20_3,5X4,5
- added C1, C10, C11, C12, C2, C9: 10uF, SparkFun-Capacitors:0402-CAP
- added C3, C4: 400uF, SparkFun-Capacitors:PANASONIC_G
- added C5: 22pF, SparkFun-Capacitors:0402-CAP
- added C6: 4.7uF, SparkFun-Capacitors:0402-CAP
- added C7, C8: 100nF, SparkFun-Capacitors:0402-CAP
- added GPS_DEBUG, LIBATRY: (no value), SparkFun-Connectors:1X03
- added IC3: CP2102, silabs:MLP28
- added JP1: USB-MICROB, SparkFun-Connectors:USB-MICROB
- added L2: 22uH, SparkFun-Passives:C0402
- added LED1, LED4: (no value), led:SML0603
- added Q1, Q2: (no value), SparkFun-DiscreteSemi:SOT23
- added R1: 0R, SparkFun-Passives:0402-RES
- added R10: 240k, SparkFun:0402-RES
- added R11, R12, R13: 22R, SparkFun:0402-RES
- added R14, R15: (no value), SparkFun-Passives:0402-RES
- added R16: (no value), SparkFun:0402-RES
- added R2, R5: 470, SparkFun-Passives:0402-RES
- added R3: 4.7k, SparkFun-Passives:0402-RES
- added R4: 47k, SparkFun-Passives:0402-RES
- added R9: 300k, SparkFun:0402-RES
- added SJ1: (no value), jumper:SJ_2
- added U$2: SIMHOLDER3, SparkFun-Connectors:SIMHOLDER3
- added U1: TPS62122_DRV_6, myTracelib:DRV6_1P6X1
- moved G1 42.0 mm to (9.16, 31.8)
- moved IC1 18.0 mm to (20.0, 18.0), turned to 180 degrees
- moved U$1 15.6 mm to (57.0, 20.1), turned to 90 degrees
Connections:
- removed net AVCC: IC1.64
- removed net AVSS: IC1.62
- removed net DVCC: IC1.1
- removed net DVSS: IC1.63
- removed net VSS: IC2.10
- new net GND: C1.1, C10.1, C11.1, C2.1, C3.-, C4.-, C6.2, C7.1, C8.1, C9.1, G1.-, GPS_DEBUG.1, IC1.11, IC1.62, IC1.63, IC3.3, IC3.EXP, IC3.M, JP1.GND, JP1.MT1, JP1.MT2, LED1.C, LIBATRY.3, Q2.2, R10.1, R4.1, U$1.P$1, U$1.P$10, U$1.P$14, U$1.P$2, U$1.P$37, U$1.P$40, U$1.P$41, U$1.P$43, U$1.P$5, U$1.P$57, U$1.P$58, U$1.P$60, U$1.P$61, U$1.P$64, U$1.P$65, U$1.P$77, U$1.P$78, U$1.P$80, U$2.6, U1.6
- new net GPS_RXD: GPS_DEBUG.2, U$1.P$16
- new net GPS_TXD: GPS_DEBUG.3, U$1.P$15
- new net GSM_CTS: IC1.13, U$1.P$67
- new net GSM_DCD: IC1.14, U$1.P$70
- new net GSM_DTR: IC1.16, U$1.P$72
- new net GSM_PWRKEY: IC1.18, R3.2
- new net GSM_RI: IC1.15, U$1.P$69
- new net GSM_RTS: IC1.12, U$1.P$66
- new net GSM_STATUS: IC1.17, U$1.P$52
- new net N$10: R11.1, U$2.2
- new net N$11: C2.2, IC3.6
- new net N$12: L2.1, U1.1
- new net N$14: C11.2, SJ1.2
- new net N$15: IC3.7, IC3.8, IC3.9, R1.2, R2.2
- new net N$16: R12.1, U$2.3
- new net N$17: R13.2, U$2.4
- new net N$19: C5.2, R10.2, R9.1, U1.3
- new net N$2: IC1.7, SJ1.1
- new net N$21: C12.2, IC3.28
- new net N$23: Q1.2, R15.1
- new net N$24: Q1.1, R14.2, R15.2
- new net N$25: IC1.19
- new net N$4: LED4.C, Q1.3
- new net N$5: LED1.A, R2.1
- new net N$7: LED4.A, R16.1
- new net N$8: Q2.1, R3.1, R4.2
- new net NETL: R14.1, U$1.P$51
- new net NTC: LIBATRY.2, U$1.P$73
- new net PWRKEY: Q2.3, U$1.P$3
- new net RESET: C12.1, IC1.58, R5.1
- new net SIM_CLK: R12.2, U$1.P$19
- new net SIM_DATA: C8.2, R13.1, U$1.P$17
- new net SIM_RST: R11.2, U$1.P$18
- new net SIM_VDD: C7.2, U$1.P$20, U$2.1
- new net UART0_RXD: IC1.33, IC3.26
- new net UART0_TXD: IC1.32, IC3.25
- new net UART1_RXD: IC1.35, U$1.P$71
- new net UART1_TXD: IC1.34, U$1.P$68
- new net USB_N: IC3.5, JP1.D-
- new net USB_P: IC3.4, JP1.D+
- new net VBAT: C3.+, C4.+, LIBATRY.1, R16.2, U$1.P$62, U$1.P$63, U1.4, U1.5
- new net VBUS: C1.2, JP1.VBUS, R1.1, U$1.P$74
- new net VDD: C10.2, C5.1, C6.1, C9.2, IC1.1, IC1.10, IC1.64, L2.2, R5.2, R9.2, U1.2
- new net VRTC: G1.+@1, G1.+@2, U$1.P$42
Other:
- board size 88.6 x 63.5 mm -> 75.9 x 38.1 mm

Commit message: normal Push.
Parts:
- added LED2: (no value), led:SML0603
- added PROG: (no value), SparkFun-Connectors:1X06_SMD_STRAIGHT
- added R6, R7: 1k, SparkFun-Passives:0402-RES
- added R8: (no value), SparkFun:0402-RES
- GPS_DEBUG: value (none) -> 1x3 RA Female .1"; device SparkFun-Connectors:1X03 -> SparkFun-Connectors:1X03_SMD_RA_FEMALE
- moved GPS_DEBUG 23.9 mm to (44.1, -5.05), flipped to the bottom, turned to 0 degrees
- moved G1 23.6 mm to (8.86, 8.18), flipped to the bottom, turned to 180 degrees
- moved C2 4.57 mm to (2.04, 16.7)
- moved R2 4.18 mm to (2.76, 29.1)
- moved R1 3.05 mm to (7.95, 23.2)
- moved Q2 2.76 mm to (39.7, 6.74)
- moved R4 2.29 mm to (35.0, 5.29)
- moved R3 1.98 mm to (35.0, 6.98)
- moved C12 1.92 mm to (7.97, 14.6), turned to 90 degrees
- moved R10 1.70 mm to (21.1, 4.69), turned to 270 degrees
- moved C11 1.52 mm to (18.5, 31.0)
- moved LED1 1.10 mm to (2.91, 27.6)
- moved U1 0.93 mm to (16.9, 4.15)
- moved R9 0.57 mm to (21.1, 1.56), turned to 270 degrees
- moved R5 0.46 mm to (28.0, 17.5)
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Connections:
- new net N$1: IC1.57, PROG.1
- new net N$13: LED2.A, R8.1
- new net N$20: IC1.59, R6.1, R7.2
- new net N$3: IC1.55, PROG.2
- new net N$6: IC1.54, PROG.3
- new net N$9: IC1.56, PROG.4
- net GND: now also PROG.6, R7.1, U1.7
- net N$25: now also R8.2
- net RESET: now also PROG.5
- net VBAT: now also R6.2
- net VDD: now also LED2.C
Routing:
- net GND: track 0.00 -> 359.0 mm, vias 0 -> 20
- net VRTC: track 0.00 -> 97.2 mm, vias 0 -> 1
- net VDD: track 0.00 -> 95.7 mm, vias 0 -> 8
- net VBAT: track 0.00 -> 91.6 mm, vias 0 -> 5
- net RESET: track 0.00 -> 72.4 mm, vias 0 -> 1
- net SIM_DATA: track 0.00 -> 69.6 mm, vias 0 -> 1
- net GSM_STATUS: track 0.00 -> 64.3 mm, vias 0 -> 2
- net VBUS: track 0.00 -> 57.1 mm, vias 0 -> 5
- net NTC: track 0.00 -> 53.8 mm, vias 0 -> 3
- net SIM_VDD: track 0.00 -> 50.3 mm, vias 0 -> 1
- net UART1_TXD: track 0.00 -> 41.2 mm, vias 0 -> 2
- net SIM_RST: track 0.00 -> 40.6 mm, vias 0 -> 1
- net UART1_RXD: track 0.00 -> 38.2 mm, vias 0 -> 2
- net SIM_CLK: track 0.00 -> 37.8 mm, vias 0 -> 1
- net GSM_DTR: track 0.00 -> 37.7 mm, vias 0 -> 2
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- added copper zone on layer 1, net GND
- added copper zone on layer 16, net GND

Commit message: normal push
Other:
- board size 75.9 x 38.1 mm -> 76.2 x 38.1 mm
