File: boardFiles/BoardVariant/solution/schematic.sch (EAGLE design)
At the start: 4 parts, among them IC1 MSP430F1491, IC2 BQ24120

Commit message: Normal Push.
Parts:
- removed IC2: BQ24120, texas:BQ24120
- added C1, C10, C11, C12, C2, C9: 10uF, SparkFun-Capacitors:CAP0402-CAP
- added C3, C4: 400uF, SparkFun-Capacitors:CAP_POLG
- added C5: 22pF, SparkFun-Capacitors:CAP0402-CAP
- added C6: 4.7uF, SparkFun-Capacitors:CAP0402-CAP
- added C7, C8: 100nF, SparkFun-Capacitors:CAP0402-CAP
- added GPS_DEBUG, LIBATRY: (no value), SparkFun-Connectors:M03PTH
- added IC3: CP2102, silabs:CP2102
- added JP1: USB-MICROB, SparkFun-Connectors:USB-MICROB
- added L2: 22uH, SparkFun-Passives:INDUCTOR0402
- added LED1, LED4: (no value), led:LEDSML0603
- added Q1, Q2: (no value), SparkFun-DiscreteSemi:TRANSISTOR_NPNSOT23
- added R1: 0R, SparkFun-Passives:RESISTOR0402-RES
- added R10: 240k, SparkFun:RESISTOR0402-RES
- added R11, R12, R13: 22R, SparkFun:RESISTOR0402-RES
- added R14, R15: (no value), SparkFun-Passives:RESISTOR0402-RES
- added R16: (no value), SparkFun:RESISTOR0402-RES
- added R2, R5: 470, SparkFun-Passives:RESISTOR0402-RES
- added R3: 4.7k, SparkFun-Passives:RESISTOR0402-RES
- added R4: 47k, SparkFun-Passives:RESISTOR0402-RES
- added R9: 300k, SparkFun:RESISTOR0402-RES
- added SJ1: (no value), jumper:SJ2W
- added U$2: SIMHOLDER3, SparkFun-Connectors:SIMHOLDER3
- added U1: TPS62122_DRV_6, myTracelib:TPS62122_DRV_6
Connections:
- new net GND: C1.1, C10.1, C11.1, C2.1, C3.-, C4.-, C6.2, C7.1, C8.1, C9.1, G1.-, GPS_DEBUG.1, IC1.AVSS, IC1.DVSS, IC1.VREF-/VEREF-, IC3.GND, IC3.GND@EXP, IC3.GND@M, JP1.GND, LED1.C, LIBATRY.3, Q2.E, R10.1, R4.1, U$1.GND1, U$1.GND10, U$1.GND11, U$1.GND12, U$1.GND13, U$1.GND14, U$1.GND15, U$1.GND16, U$1.GND17, U$1.GND18, U$1.GND2, U$1.GND3, U$1.GND4, U$1.GND5, U$1.GND6, U$1.GND7, U$1.GND8, U$1.GND9, U$2.GND, U1.GND
- new net GPS_RXD: GPS_DEBUG.2, U$1.GPSDRXD
- new net GPS_TXD: GPS_DEBUG.3, U$1.GPSDTXD
- new net GSM_CTS: IC1.P1.1, U$1.CTS
- new net GSM_DCD: IC1.P1.2, U$1.DCD
- new net GSM_DTR: IC1.P1.4, U$1.DTR
- new net GSM_PWRKEY: IC1.P1.6, R3.2
- new net GSM_RI: IC1.P1.3, U$1.RI
- new net GSM_RTS: IC1.P1.0, U$1.RTS
- new net GSM_STATUS: IC1.P1.5, U$1.STATUS
- new net N$10: R11.1, U$2.RST
- new net N$11: C2.2, IC3.VDD
- new net N$12: L2.1, U1.SW
- new net N$14: C11.2, SJ1.2
- new net N$15: IC3.!RST, IC3.REGIN, IC3.VBUS, R1.2, R2.2
- new net N$16: R12.1, U$2.CLK
- new net N$17: R13.2, U$2.I/O
- new net N$19: C5.2, R10.2, R9.1, U1.FB
- new net N$2: IC1.VREF+, SJ1.1
- new net N$21: C12.2, IC3.DTR
- new net N$23: Q1.E, R15.1
- new net N$24: Q1.B, R14.2, R15.2
- new net N$25: IC1.P1.7
- new net N$4: LED4.C, Q1.C
- new net N$5: LED1.A, R2.1
- new net N$7: LED4.A, R16.1
- new net N$8: Q2.B, R3.1, R4.2
- new net NETL: R14.1, U$1.NETLGHT
- new net NTC: LIBATRY.2, U$1.TEMP_BAT
- new net PWRKEY: Q2.C, U$1.PWRKEY
- new net RESET: C12.1, IC1.!RTS!/NMI, R5.1
- new net SIM_CLK: R12.2, U$1.SIMCLK
- new net SIM_DATA: C8.2, R13.1, U$1.SIMDATA
- new net SIM_RST: R11.2, U$1.SIMRST
- new net SIM_VDD: C7.2, U$1.SIMVDD, U$2.VCC
- new net UART0_RXD: IC1.P3.5, IC3.TXD
- new net UART0_TXD: IC1.P3.4, IC3.RXD
- new net UART1_RXD: IC1.P3.7, U$1.TXD
- new net UART1_TXD: IC1.P3.6, U$1.RXD
- new net USB_N: IC3.D-, JP1.D-
- new net USB_P: IC3.D+, JP1.D+
- new net VBAT: C3.+, C4.+, LIBATRY.1, R16.2, U$1.VBAT1, U$1.VBAT2, U1.EN, U1.VIN
- new net VBUS: C1.2, JP1.VBUS, R1.1, U$1.VCHG
- new net VDD: C10.2, C5.1, C6.1, C9.2, IC1.AVCC, IC1.DVCC, IC1.VEREF+, L2.2, R5.2, R9.2, U1.VOUT
- new net VRTC: G1.+, U$1.VRTC
Other:
- moved on the sheet: G1, IC1, U$1

Commit message: normal Push.
Parts:
- added LED2: (no value), led:LEDSML0603
- added PROG: (no value), SparkFun-Connectors:M06SMD-STRAIGHT
- added R6, R7: 1k, SparkFun-Passives:RESISTOR0402-RES
- added R8: (no value), SparkFun:RESISTOR0402-RES
- GPS_DEBUG: value (none) -> 1x3 RA Female .1"; device SparkFun-Connectors:M03PTH -> SparkFun-Connectors:M03SMD_RA_FEMALE
Connections:
- new net N$1: IC1.TCK, PROG.1
- new net N$13: LED2.A, R8.1
- new net N$20: IC1.P6.0, R6.1, R7.2
- new net N$3: IC1.TDI, PROG.2
- new net N$6: IC1.TDO/TDI, PROG.3
- new net N$9: IC1.TMS, PROG.4
- net GND: now also PROG.6, R7.1, U1.EPAD
- net N$25: now also R8.2
- net RESET: now also PROG.5
- net VBAT: now also R6.2
- net VDD: now also LED2.C
Other:
- note added: "Battery"
- note added: "CP2102"
- note added: "MSP430F1491"
- note added: "SIM908"
- note added: "Sim Card"
- note added: "Switching Regulator"
- note added: "USB"
- moved on the sheet: C1, C10, C11, C12, C2, C3, C4, C5, C6, C7, C8, C9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
